Commit message: urdf file changes

File: src/columbusmaximus/description/robot_core.xacro (robot description, xacro)
@@ -1,5 +1,4 @@
 <?xml version="1.0"?>
 <robot name="columbusmaximus" xmlns:xacro="http://www.ros.org/wiki/xacro">
-  <!-- ===== Properties ===== -->
   <xacro:property name="wheel_radius" value="0.05"/>
   <xacro:property name="wheel_length" value="0.04"/>
@@ -10,7 +9,5 @@
   <xacro:property name="caster_offset_x" value="0.15"/>
   <xacro:property name="caster_offset_z" value="-0.08"/>
-  <!-- ===== base_link: empty reference frame ===== -->
   <link name="base_link"></link>
-  <!-- ===== Fixed joint: base_link -> chassis ===== -->
   <joint name="chassis_joint" type="fixed">
     <parent link="base_link"/>
@@ -18,5 +15,4 @@
     <origin xyz="0 0 0" rpy="0 0 0"/>
   </joint>
-  <!-- ===== chassis: your STL mesh lives here ===== -->
   <link name="chassis">
     <visual>
@@ -40,62 +36,3 @@
     </inertial>
   </link>
-  <!-- ===== Drive wheel macro (left + right, continuous joints, attached to chassis) ===== -->
-  <xacro:macro name="drive_wheel" params="prefix y_offset">
-    <link name="${prefix}_wheel">
-      <visual>
-        <geometry>
-          <cylinder radius="${wheel_radius}" length="${wheel_length}"/>
-        </geometry>
-        <material name="black">
-          <color rgba="0.1 0.1 0.1 1"/>
-        </material>
-      </visual>
-      <collision>
-        <geometry>
-          <cylinder radius="${wheel_radius}" length="${wheel_length}"/>
-        </geometry>
-      </collision>
-      <inertial>
-        <mass value="0.05"/>
-        <origin xyz="0 0 0" rpy="0 0 0"/>
-        <inertia ixx="0.00002708" ixy="0.0" ixz="0.0"
-                 iyy="0.00002708" iyz="0.0" izz="0.0000625"/>
-      </inertial>
-    </link>
-    <joint name="chassis_to_${prefix}_wheel" type="continuous">
-      <parent link="chassis"/>
-      <child link="${prefix}_wheel"/>
-      <origin xyz="${wheel_offset_x} ${y_offset} ${wheel_offset_z}" rpy="1.5708 0 0"/>
-      <axis xyz="0 0 1"/>
-    </joint>
-  </xacro:macro>
-  <xacro:drive_wheel prefix="left"  y_offset="${wheel_offset_y}"/>
-  <xacro:drive_wheel prefix="right" y_offset="${-wheel_offset_y}"/>
-  <!-- ===== Caster wheel (passive, attached to chassis) ===== -->
-  <link name="caster_wheel">
-    <visual>
-      <geometry>
-        <sphere radius="${caster_radius}"/>
-      </geometry>
-      <material name="black">
-        <color rgba="0.1 0.1 0.1 1"/>
-      </material>
-    </visual>
-    <collision>
-      <geometry>
-        <sphere radius="${caster_radius}"/>
-      </geometry>
-    </collision>
-    <inertial>
-      <mass value="0.02"/>
-      <origin xyz="0 0 0" rpy="0 0 0"/>
-      <inertia ixx="0.0000032" ixy="0.0" ixz="0.0"
-               iyy="0.0000032" iyz="0.0" izz="0.0000032"/>
-    </inertial>
-  </link>
-  <joint name="chassis_to_caster_wheel" type="fixed">
-    <parent link="chassis"/>
-    <child link="caster_wheel"/>
-    <origin xyz="${caster_offset_x} 0 ${caster_offset_z}" rpy="0 0 0"/>
-  </joint>
 </robot>

Commit message: Added wheels to urdf model

File: src/columbusmaximus/description/robot_core.xacro (robot description, xacro)
@@ -1,20 +1,16 @@
 <?xml version="1.0"?>
 <robot name="columbusmaximus" xmlns:xacro="http://www.ros.org/wiki/xacro">
-  <xacro:property name="wheel_radius" value="0.05"/>
-  <xacro:property name="wheel_length" value="0.04"/>
-  <xacro:property name="wheel_offset_x" value="-0.10"/>
-  <xacro:property name="wheel_offset_y" value="0.18"/>
-  <xacro:property name="wheel_offset_z" value="-0.05"/>
   <xacro:property name="caster_radius" value="0.02"/>
-  <xacro:property name="caster_offset_x" value="0.15"/>
-  <xacro:property name="caster_offset_z" value="-0.08"/>
+  <xacro:property name="caster_offset_x" value="0.12"/>
+  <xacro:property name="caster_offset_z" value="-0.02"/>
   <link name="base_link"></link>
   <joint name="chassis_joint" type="fixed">
     <parent link="base_link"/>
     <child link="chassis"/>
-    <origin xyz="0 0 0" rpy="0 0 0"/>
+    <origin xyz="0.0575 0 0" rpy="0 0 0"/>
   </joint>
   <link name="chassis">
     <visual>
+      <origin xyz="0.07193 -0.01172 0" rpy="0 0 ${pi/2}"/>
       <geometry>
         <mesh filename="package://columbusmaximus/meshes/Assembly_1.stl" scale="0.001 0.001 0.001"/>
@@ -25,4 +21,5 @@
     </visual>
     <collision>
+      <origin xyz="0.07193 -0.01172 0" rpy="0 0 ${pi/2}"/>
       <geometry>
         <mesh filename="package://columbusmaximus/meshes/Assembly_1.stl" scale="0.001 0.001 0.001"/>
@@ -36,3 +33,86 @@
     </inertial>
   </link>
+  <!-- ===== Left wheel===== -->
+  <link name="left_wheel">
+    <visual>
+      <geometry>
+        <cylinder radius="0.04" length="0.04"/>
+      </geometry>
+      <material name="black">
+        <color rgba="0.1 0.1 0.1 1"/>
+      </material>
+    </visual>
+    <collision>
+      <geometry>
+        <cylinder radius="0.04" length="0.04"/>
+      </geometry>
+    </collision>
+    <inertial>
+      <mass value="0.05"/>
+      <origin xyz="0 0 0" rpy="0 0 0"/>
+      <inertia ixx="0.00002708" ixy="0.0" ixz="0.0"
+               iyy="0.00002708" iyz="0.0" izz="0.0000625"/>
+    </inertial>
+  </link>
+  <joint name="chassis_to_left_wheel" type="continuous">
+    <parent link="chassis"/>
+    <child link="left_wheel"/>
+    <origin xyz="0 0.122 0" rpy="1.5708 0 0"/>
+    <axis xyz="0 0 1"/>
+  </joint>
+  <!-- ===== Right wheel===== -->
+  <link name="right_wheel">
+    <visual>
+      <geometry>
+        <cylinder radius="0.04" length="0.04"/>
+      </geometry>
+      <material name="black">
+        <color rgba="0.1 0.1 0.1 1"/>
+      </material>
+    </visual>
+    <collision>
+      <geometry>
+        <cylinder radius="0.04" length="0.04"/>
+      </geometry>
+    </collision>
+    <inertial>
+      <mass value="0.05"/>
+      <origin xyz="0 0 0" rpy="0 0 0"/>
+      <inertia ixx="0.00002708" ixy="0.0" ixz="0.0"
+               iyy="0.00002708" iyz="0.0" izz="0.0000625"/>
+    </inertial>
+  </link>
+  <joint name="chassis_to_right_wheel" type="continuous">
+    <parent link="chassis"/>
+    <child link="right_wheel"/>
+    <origin xyz="0 -0.122 0" rpy="1.5708 0 0"/>
+    <axis xyz="0 0 1"/>
+  </joint>
+  <!-- ===== Caster wheel===== -->
+  <link name="caster_wheel">
+    <visual>
+      <geometry>
+        <sphere radius="${caster_radius}"/>
+      </geometry>
+      <material name="black">
+        <color rgba="0.1 0.1 0.1 1"/>
+      </material>
+    </visual>
+    <collision>
+      <geometry>
+        <sphere radius="${caster_radius}"/>
+      </geometry>
+    </collision>
+    <inertial>
+      <mass value="0.02"/>
+      <origin xyz="0 0 0" rpy="0 0 0"/>
+      <inertia ixx="0.0000032" ixy="0.0" ixz="0.0"
+               iyy="0.0000032" iyz="0.0" izz="0.0000032"/>
+    </inertial>
+  </link>
+  <joint name="chassis_to_caster_wheel" type="fixed">
+    <parent link="chassis"/>
+    <child link="caster_wheel"/>
+    <origin xyz="${caster_offset_x} 0 ${caster_offset_z}" rpy="0 0 0"/>
+  </joint>
 </robot>

Commit message: Gazebo rendering and teleop

File: src/columbusmaximus/description/robot_core.xacro (robot description, xacro)
@@ -24,4 +24,5 @@
       <geometry>
         <mesh filename="package://columbusmaximus/meshes/Assembly_1.stl" scale="0.001 0.001 0.001"/>
+        <!--<box size="0.216 0.268 0.2"/>-->
       </geometry>
     </collision>
@@ -58,5 +59,5 @@
     <parent link="chassis"/>
     <child link="left_wheel"/>
-    <origin xyz="0 0.122 0" rpy="1.5708 0 0"/>
+    <origin xyz="0 0.122 0" rpy="-1.5708 0 0"/>
     <axis xyz="0 0 1"/>
   </joint>
@@ -87,5 +88,5 @@
     <child link="right_wheel"/>
     <origin xyz="0 -0.122 0" rpy="1.5708 0 0"/>
-    <axis xyz="0 0 1"/>
+    <axis xyz="0 0 -1"/>
   </joint>
   <!-- ===== Caster wheel===== -->
@@ -116,3 +117,7 @@
     <origin xyz="${caster_offset_x} 0 ${caster_offset_z}" rpy="0 0 0"/>
   </joint>
+  <gazebo reference="caster_wheel">
+    <mu1>0.001</mu1>
+    <mu2>0.001</mu2>
+   </gazebo>
 </robot>

Commit message: Integration of lidar sensor

File: src/columbusmaximus/description/robot_core.xacro (robot description, xacro)
@@ -4,4 +4,16 @@
   <xacro:property name="caster_offset_x" value="0.12"/>
   <xacro:property name="caster_offset_z" value="-0.02"/>
+  <material name="black">
+    <color rgba="0 0 0 1"/>
+  </material>
+   <material name="blue">
+    <color rgba="0 0 1 1"/>
+  </material>
+   <material name="red ">
+    <color rgba="1 0 0 1"/>
+  </material>
+  <material name="grey ">
+    <color rgba="0.6 0.6 0.6 1"/>
+  </material>
   <link name="base_link"></link>
   <joint name="chassis_joint" type="fixed">
@@ -34,4 +46,7 @@
     </inertial>
   </link>
+  <gazebo reference="chassis">
+    <material>Gazebo/Grey</material>
+  </gazebo>
   <!-- ===== Left wheel===== -->
   <link name="left_wheel">
@@ -62,4 +77,7 @@
     <axis xyz="0 0 1"/>
   </joint>
+  <gazebo reference="left_wheel">
+    <material>Gazebo/Black</material>
+  </gazebo>
   <!-- ===== Right wheel===== -->
   <link name="right_wheel">
@@ -90,4 +108,7 @@
     <axis xyz="0 0 -1"/>
   </joint>
+  <gazebo reference="right_wheel">
+    <material>Gazebo/Black</material>
+  </gazebo>
   <!-- ===== Caster wheel===== -->
   <link name="caster_wheel">
@@ -120,4 +141,5 @@
     <mu1>0.001</mu1>
     <mu2>0.001</mu2>
+    <material>Gazebo/Black</material>
    </gazebo>
 </robot>
