Commit message: Added Slam toolbox functionality

File: src/columbusmaximus/description/lidar.xacro (robot description, xacro)
@@ -26,5 +26,5 @@
             <pose>0 0 0 0 0 0</pose>
             <visualize>true</visualize>
-            <update_rate>10</update_rate>
+            <update_rate>5</update_rate>
             <ray>
                 <scan>

File: src/columbusmaximus/description/robot_core.xacro (robot description, xacro)
@@ -108,4 +108,11 @@
     <axis xyz="0 0 -1"/>
   </joint>
+  <joint name = "base_footprint_joint" type="fixed">
+    <parent link="base_link"/>
+    <child link="base_footprint"/>
+    <origin xyz="0 0 0" rpy="0 0 0"/>
+  </joint>
+  <link name="base_footprint">
+   </link>
   <gazebo reference="right_wheel">
     <material>Gazebo/Black</material>
@@ -127,5 +134,5 @@
     </collision>
     <inertial>
-      <mass value="0.02"/>
+      <mass value="0.5"/>
       <origin xyz="0 0 0" rpy="0 0 0"/>
       <inertia ixx="0.0000032" ixy="0.0" ixz="0.0"
